File: apple2-slot-riser.kicad_pcb (KiCad board)
At the start: 2 copper layers, 89.9 x 50.8 mm, 6 parts, among them J1 CARD EDGE, J2 STRADDLE MOUNT, J3 RIGHT ANGLE, J4 EXTENDER / LOGIC ANALYZER

Commit message: Add modified Kicad Files and Gerber
Parts:
- removed J3: RIGHT ANGLE, footprint:CardEdge_EDEC_3x5-050_2x25_P2.54mm_CCW
- removed J4: EXTENDER / LOGIC ANALYZER, footprint:IDC-Header_2x25_P2.54mm_Vertical_CCW
- J2: value STRADDLE MOUNT -> *** DANGER Flipped connector for F/F Ribbon Cable ***
Connections:
- J1 pad 34: Net-(J1-Pad34) -> -5V
- J1 pad 50: Net-(J1-Pad50) -> -12V
- J2 pad 33: Net-(J2-Pad33) -> Net-(J1-Pad33)
- J2 pad 34: Net-(J2-Pad34) -> -5V
- J2 pad 50: Net-(J2-Pad50) -> -12V
Routing:
- net -5V: track 0.00 -> 44.7 mm, vias 0 -> 1
- net Net-(J1-Pad33): track 0.00 -> 44.2 mm, vias 0 -> 1
- net -12V: track 0.00 -> 44.2 mm, vias 0 -> 1
- net +5V: track 52.3 -> 57.2 mm, vias 0 -> 4
- net /DMA: track 45.3 -> 43.2 mm, vias 0 -> 1
- net /RW: track 45.3 -> 43.2 mm, vias 0 -> 1
- net /A9: track 45.3 -> 43.2 mm, vias 0 -> 1
- net /A3: track 45.3 -> 43.2 mm, vias 0 -> 1
- net /A1: track 45.3 -> 43.2 mm, vias 0 -> 1
- net /IOSEL: track 45.3 -> 43.2 mm, vias 0 -> 1
- net /RDY: track 45.3 -> 43.2 mm, vias 0 -> 1
- net /NC19: track 45.3 -> 43.2 mm, vias 0 -> 1
- net /IOSTROBE: track 45.3 -> 43.2 mm, vias 0 -> 1
- net /INT_OUT: track 45.3 -> 43.2 mm, vias 0 -> 1
- net /DMA_OUT: track 45.3 -> 43.2 mm, vias 0 -> 1
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Other:
- outline, holes or cut-outs redrawn
- net class Default removed
- net class Power removed
- board text added: "*** DANGER Flipped connector for F/F Ribbon Cable ***"
- board text added: "APPLE II CARD ADAPTER"
- board text added: "DANGER +12V, -12V, -5V IS CONNECTED!"
- board text added: "back →"
- board text added: "rev 0 2025/03/11 www.mrtechgadget.com"
- board text added: "← motherboard"
- board text removed: "+12V, -12V, -5V NOT CONNECTED!"
- board text removed: "APPLE II CARD RISER"
- board text removed: "JLCJLCJLCJLC"
- board text removed: "rev 0 2020/04/24 www.reneeharke.com"
